File: ebus2usb.kicad_sch (KiCad schematic)
At the start: 55 parts, among them J1 MSTBA 2,5/2-G-5,08, J2 Molex 53047-0210, J21 TC2030, J3 Molex 53047-0410, J5 HRO TYPE-C-31-M-12, J6 Molex 53047-0210, J7 Molex 53047-0410, J8 Harwin M50-3530242, Q1 BC817-40, Q2 BC817-40, U1 AZV3002, U2 ADuM1201, U21 XC6206P332MR, U5 SRV05-4, U7 STM32L412KBT6

Commit message: Added info for TC2030-NL to schematic and BOM
Other:
- note added: "Tag-Connect 6-Pin "No Legs" TC2030-NL Plug-of-Nails"
- note removed: "[Alternatives] CH340N: CH330N"
Changed lines of the file:
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@@
     (effects (font (size 1.27 1.27)) (justify left bottom))
   )
-  (text "[Alternatives] CH340N: CH330N\n" (at 318.77 201.93 0)
+  (text "Tag-Connect \n6-Pin \"No Legs\"\nTC2030-NL \nPlug-of-Nails\n"
+    (at 208.28 193.04 0)
     (effects (font (size 1.27 1.27) (color 132 132 132 1)) (justify left bottom))
   )
